File: mainboard/mainboard.kicad_pcb (KiCad board)
At the start: 2 copper layers, 11 parts, among them J1 DISPLAY, J2 EXT1, J3 EXT3, J4 EXT2, Q1 2N7002

Commit message: mainboard finished
Parts:
- added C1: 0,1, Capacitor_SMD:C_0805_2012Metric_Pad1.15x1.40mm_HandSolder, B.Cu at (80.0, 25.0)
- added C10: 0,1, Capacitor_SMD:C_0805_2012Metric_Pad1.15x1.40mm_HandSolder, B.Cu at (91.0, 46.0)
- added C11: 0,1, Capacitor_SMD:C_0805_2012Metric_Pad1.15x1.40mm_HandSolder, B.Cu at (14.0, 64.0)
- added C12: 0,1, Capacitor_SMD:C_0805_2012Metric_Pad1.15x1.40mm_HandSolder, B.Cu at (15.0, 47.5)
- added C14: 0,1, Capacitor_SMD:C_0805_2012Metric_Pad1.15x1.40mm_HandSolder, B.Cu at (14.5, 43.0)
- added C15: 0,1, Capacitor_SMD:C_0805_2012Metric_Pad1.15x1.40mm_HandSolder, B.Cu at (7.03, 52.0)
- added C16: 0,1, Capacitor_SMD:C_0805_2012Metric_Pad1.15x1.40mm_HandSolder, B.Cu at (15.0, 12.0)
- added C2: 0,1, Capacitor_SMD:C_0805_2012Metric_Pad1.15x1.40mm_HandSolder, B.Cu at (77.0, 52.2)
- added C3: 0,1, Capacitor_SMD:C_0805_2012Metric_Pad1.15x1.40mm_HandSolder, B.Cu at (79.6, 61.0)
- added C4: 0,1, Capacitor_SMD:C_0805_2012Metric_Pad1.15x1.40mm_HandSolder, B.Cu at (86.5, 25.0)
- added C5: 0,1, Capacitor_SMD:C_0805_2012Metric_Pad1.15x1.40mm_HandSolder, B.Cu at (31.0, 61.0)
- added C6: 0,1, Capacitor_SMD:C_0805_2012Metric_Pad1.15x1.40mm_HandSolder, B.Cu at (44.0, 61.0)
- added C7: 0,1, Capacitor_SMD:C_0805_2012Metric_Pad1.15x1.40mm_HandSolder, B.Cu at (62.0, 61.0)
- added C8: 0,1, Capacitor_SMD:C_0805_2012Metric_Pad1.15x1.40mm_HandSolder, B.Cu at (77.0, 61.0)
- added C9: 0,1, Capacitor_SMD:C_0805_2012Metric_Pad1.15x1.40mm_HandSolder, B.Cu at (91.0, 27.0)
- added D1: P82B715, Package_SO:SOIC-8_3.9x4.9mm_P1.27mm, B.Cu at (73.0, 54.0)
- added J1: Conn_02x05_Odd_Even, Connector_IDC:IDC-Header_2x05_P2.54mm_Vertical, B.Cu at (14.0, 55.6)
- added J10: Conn_01x05, Connector_PinHeader_2.54mm:PinHeader_1x05_P2.54mm_Horizontal, B.Cu at (95.0, 27.0)
- added J11: Conn_01x05, Connector_PinHeader_2.54mm:PinHeader_1x05_P2.54mm_Horizontal, B.Cu at (95.0, 46.0)
- added J12: Conn_01x05, Connector_PinHeader_2.54mm:PinHeader_1x05_P2.54mm_Vertical, B.Cu at (21.6, 29.6)
- added J13: EXT3out, Connector_PinHeader_2.54mm:PinHeader_1x16_P2.54mm_Vertical, B.Cu at (5.00, 49.1)
- added J14: Conn_01x01, Connector_Wire:SolderWirePad_1x01_Drill2mm, F.Cu at (0.00, 50.0)
- added J15: Conn_01x01, Connector_Wire:SolderWirePad_1x01_Drill2mm, F.Cu at (0.00, 10.0)
- added J16: Conn_01x04, Connector_PinHeader_2.54mm:PinHeader_1x04_P2.54mm_Vertical, B.Cu at (66.2, 18.0)
- added J5: Conn_02x05_Odd_Even, Connector_IDC:IDC-Header_2x05_P2.54mm_Vertical, B.Cu at (65.0, 35.4)
- added J6: Conn_01x05, Connector_PinHeader_2.54mm:PinHeader_1x05_P2.54mm_Horizontal, B.Cu at (77.0, 65.0)
- added J7: Conn_01x05, Connector_PinHeader_2.54mm:PinHeader_1x05_P2.54mm_Horizontal, B.Cu at (23.0, 65.0)
- added J8: Conn_01x05, Connector_PinHeader_2.54mm:PinHeader_1x05_P2.54mm_Horizontal, B.Cu at (41.0, 65.0)
- added J9: Conn_01x05, Connector_PinHeader_2.54mm:PinHeader_1x05_P2.54mm_Horizontal, B.Cu at (59.0, 65.0)
- added R1: 510, Resistor_SMD:R_0805_2012Metric_Pad1.15x1.40mm_HandSolder, B.Cu at (84.8, 61.0)
- added R2: 510, Resistor_SMD:R_0805_2012Metric_Pad1.15x1.40mm_HandSolder, B.Cu at (82.2, 61.0)
- added R3: 10k, Resistor_SMD:R_0805_2012Metric_Pad1.15x1.40mm_HandSolder, B.Cu at (28.0, 6.50)
- added R4: 200k, Resistor_SMD:R_0805_2012Metric_Pad1.15x1.40mm_HandSolder, B.Cu at (89.0, 23.5)
- added R5: 5,1k, Resistor_SMD:R_0805_2012Metric_Pad1.15x1.40mm_HandSolder, B.Cu at (91.5, 23.0)
- added R6: 5,1k, Resistor_SMD:R_0805_2012Metric_Pad1.15x1.40mm_HandSolder, B.Cu at (91.5, 18.0)
- added RV1: R_POT, Potentiometer_THT:Potentiometer_Bourns_3296W_Vertical, B.Cu at (16.1, 7.00)
- added U1: PCA9306, Package_SO:SSOP-8_2.95x2.8mm_P0.65mm, B.Cu at (84.3, 20.8)
- Q1: moved to B.Cu
- U2: renamed from J1; value DISPLAY -> LCD-016N002L
- moved Q1 208.1 mm to (24.5, 6.50), turned to 180 degrees
- moved REF** 138.5 mm to (55.0, 13.0), turned to 90 degrees
- moved J4 123.0 mm to (18.6, 13.4), turned to 270 degrees
- moved REF** 98.3 mm to (55.0, 47.0), turned to 90 degrees
- moved J2 73.1 mm to (18.6, 49.0), turned to 270 degrees
- moved J3 72.1 mm to (11.0, 49.0), turned to 0 degrees
Connections:
- net Net-(J4-Pad5) renamed /button
- J2 pad 1: Net-(J2-Pad1) -> +5V
- J2 pad 2: Net-(J2-Pad2) -> GND
- J2 pad 4: Net-(J2-Pad4) -> /D-
- J2 pad 6: Net-(J2-Pad6) -> /D+
- J3 pad 1: Net-(J3-Pad1) -> +5V
- J3 pad 16: Net-(J3-Pad16) -> GND
- J3 pad 2: Net-(J3-Pad2) -> +3V3
- J4 pad 1: Net-(J4-Pad1) -> +3V3
- J4 pad 10: Net-(J4-Pad10) -> /valve5_12V
- J4 pad 11: Net-(J4-Pad11) -> /lcd_db4
- J4 pad 12: Net-(J4-Pad12) -> /i2c_rst
- J4 pad 13: Net-(J4-Pad13) -> /heat_24V
- J4 pad 14: Net-(J4-Pad14) -> /lcd_db7
- J4 pad 15: Net-(J4-Pad15) -> /lcd_rs
- J4 pad 16: Net-(J4-Pad16) -> /lcd_db6
- J4 pad 19: Net-(J4-Pad19) -> /pump_24V
- J4 pad 2: Net-(J4-Pad2) -> GND
- J4 pad 20: Net-(J4-Pad20) -> /fan_12V
- J4 pad 21: Net-(J4-Pad21) -> /reserv_24V
- J4 pad 24: Net-(J4-Pad24) -> /lcd_e
- J4 pad 26: Net-(J4-Pad26) -> /lcd_db5
- J4 pad 3: Net-(J4-Pad3) -> /SDA
- J4 pad 4: Net-(J4-Pad4) -> /SCL
- J4 pad 6: Net-(J4-Pad6) -> /valve1_12V
- J4 pad 7: Net-(J4-Pad7) -> /valve2_12V
- J4 pad 8: Net-(J4-Pad8) -> /valve3_12V
- J4 pad 9: Net-(J4-Pad9) -> /valve4_12V
- Q1 pad 1: Net-(Q1-Pad1) -> /i2c_rst
- REF** pad 1: (no net) -> GND (x2)
- U2 pad 1: Net-(J1-Pad1) -> GND
- U2 pad 11: Net-(J1-Pad11) -> /lcd_db4
- U2 pad 12: Net-(J1-Pad12) -> /lcd_db5
- U2 pad 13: Net-(J1-Pad13) -> /lcd_db6
- U2 pad 14: Net-(J1-Pad14) -> /lcd_db7
- U2 pad 15: Net-(J1-Pad15) -> +5V
- U2 pad 16: Net-(J1-Pad16) -> GND
- U2 pad 2: Net-(J1-Pad2) -> +5V
- U2 pad 4: Net-(J1-Pad4) -> /lcd_rs
- U2 pad 5: Net-(J1-Pad5) -> GND
- U2 pad 6: Net-(J1-Pad6) -> /lcd_e
Routing:
- net +5V: track 0.00 -> 292.6 mm, vias 0 -> 1
- net GND: track 0.00 -> 266.9 mm, vias 0 -> 21
- net +3V3: track 0.00 -> 232.6 mm, vias 0 -> 2
- net /SCL: track 0.00 -> 182.0 mm, vias 0 -> 2
- net /SDA: track 0.00 -> 173.9 mm, vias 0 -> 2
- net /fan_12V: track 0.00 -> 63.5 mm, vias 0 -> 2
- net /valve5_12V: track 0.00 -> 59.3 mm, vias 0 -> 2
- net /valve1_12V: track 0.00 -> 59.1 mm, vias 0 -> 2
- net /valve3_12V: track 0.00 -> 58.5 mm, vias 0 -> 2
- net /heat_24V: track 0.00 -> 56.7 mm, vias 0 -> 2
- net /valve4_12V: track 0.00 -> 55.3 mm, vias 0 -> 2
- net /valve2_12V: track 0.00 -> 54.7 mm, vias 0 -> 2
- net /reserv_24V: track 0.00 -> 54.3 mm, vias 0 -> 2
- net /pump_24V: track 0.00 -> 51.9 mm, vias 0 -> 2
- net Net-(J12-Pad2): track 0.00 -> 46.5 mm, vias 0 -> 1
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- added copper zone on F.Cu, net GND
Other:
- board outline added: 104 x 72 mm
