File: mainboard/mainboard.sch (KiCad schematic (older format))
At the start: 29 parts

Commit message: mainboard: work in progress
Parts:
- added C? (x5): 0,1, Capacitor_SMD:C_0805_2012Metric_Pad1.15x1.40mm_HandSolder, symbol Device:C
- added J1: DISPLAY, Connector_PinHeader_2.54mm:PinHeader_1x16_P2.54mm_Vertical, symbol Connector_Generic:Conn_01x16
- added J?: Conn_02x05_Odd_Even, symbol Connector_Generic:Conn_02x05_Odd_Even
- added J?: USB_A, symbol Connector:USB_A
- added RV1: R_POT, symbol Device:R_POT
- C1, C10, C2, C3, C4, C5, C6, C7, C8, C9: renamed from C?; footprint (none) -> Capacitor_SMD:C_0805_2012Metric_Pad1.15x1.40mm_HandSolder
- D1: renamed from D?; footprint (none) -> Package_SO:SOIC-8_3.9x4.9mm_P1.27mm
- J10, J11, J6, J7, J8, J9: renamed from J?; footprint (none) -> Connector_PinHeader_2.54mm:PinHeader_1x05_P2.54mm_Horizontal
- J2, J4: renamed from J?; footprint (none) -> Connector_PinSocket_2.54mm:PinSocket_2x13_P2.54mm_Vertical
- J3: renamed from J?; footprint (none) -> Connector_PinHeader_2.54mm:PinHeader_1x16_P2.54mm_Vertical
- J5: renamed from J?; footprint (none) -> Connector_IDC:IDC-Header_2x05_P2.54mm_Vertical
- Q1: renamed from Q?; footprint Package_TO_SOT_SMD:SOT-23 -> Package_TO_SOT_SMD:SOT-23_Handsoldering
- R1, R2, R3, R4, R5, R6: renamed from R?; footprint (none) -> Resistor_SMD:R_0805_2012Metric_Pad1.15x1.40mm_HandSolder
- U1: renamed from U?; footprint (none) -> Package_SO:SSOP-8_2.95x2.8mm_P0.65mm
Connections:
- net +3V3: now also J3.2 (Pin_2), J4.1 (Pin_1), C?.2, C?.2
- net +5V: now also J2.1 (Pin_1), J3.1 (Pin_1), C?.2, C?.2, C?.2, J?.1 (Pin_1), J?.1 (VBUS), J?.2 (Pin_2)
- net GND: now also J2.2 (Pin_2), J3.16 (Pin_16), J4.2 (Pin_2), J5.1 (Pin_1), C?.1, C?.1, C?.1, C?.1, C?.1, J1.1 (Pin_1), J?.4 (GND), J?.7 (Pin_7), J?.8 (Pin_8), RV1.1
- net SCL: now also J4.4 (Pin_4)
- net SDA: now also J4.3 (Pin_3)
- net D-: now reaches J2.4 (Pin_4)
- net D-: now also J?.2 (D-), J?.3 (Pin_3), J?.4 (Pin_4)
- net D+: now reaches J2.6 (Pin_6)
- net D+: now also J?.3 (D+), J?.5 (Pin_5), J?.6 (Pin_6)
- net at J4.11 (Pin_11): now also J1.11 (Pin_11)
- net at J4.14 (Pin_14): now also J1.12 (Pin_12)
- net at J4.15 (Pin_15): now also J1.13 (Pin_13)
- net at J4.16 (Pin_16): now also J1.14 (Pin_14)
- net valve5_12V: now reaches J5.10 (Pin_10)
- net valve1_12V: now reaches J5.2 (Pin_2)
- net heat_24V: now reaches J5.3 (Pin_3)
- net valve2_12V: now reaches J5.4 (Pin_4)
- net pump_24V: now reaches J5.5 (Pin_5)
- net valve3_12V: now reaches J5.6 (Pin_6)
- net reserv_24V: now reaches J5.7 (Pin_7)
- net valve4_12V: now reaches J5.8 (Pin_8)
- net fan_12V: now reaches J5.9 (Pin_9)
- new net: J1.2 (Pin_2), RV1.3
- new net: J1.3 (Pin_3), RV1.2
- no-connect marks 0 -> 1
Other:
- note added: "удалить"
- moved on the sheet: J2, J3, J4, J5

Commit message: fixup! mainboard: work in progress
Parts:
- removed J1: DISPLAY, Connector_PinHeader_2.54mm:PinHeader_1x16_P2.54mm_Vertical, symbol Connector_Generic:Conn_01x16
- added U?: LCD-016N002L, Display:LCD-016N002L, symbol Display_Character:LCD-016N002L
- D1: symbol k_digital_mix:P82B715 -> mainboard-rescue:P82B715-k_digital_mix
Connections:
- net +5V: now also RV1.1, U?.15 (A/VEE), U?.2 (VDD)
- net GND: now also RV1.3, U?.1 (VSS), U?.16 (K), U?.5 (R/~W); no longer RV1.1
- net fan_12V: now also J4.20 (Pin_20)
- net heat_24V: now also J4.13 (Pin_13)
- net pump_24V: now also J4.19 (Pin_19)
- net reserv_24V: now also J4.21 (Pin_21)
- net valve1_12V: now also J4.6 (Pin_6)
- net valve2_12V: now also J4.7 (Pin_7)
- net valve3_12V: now also J4.8 (Pin_8)
- net valve4_12V: now also J4.9 (Pin_9)
- net valve5_12V: now also J4.10 (Pin_10)
- net lcd_db4: now reaches J4.11 (Pin_11)
- net lcd_db4: now also U?.11 (DB4)
- net i2c_rst: now reaches J4.12 (Pin_12)
- net i2c_rst: now also Q1.1 (G), R3.1
- net lcd_db7: now reaches J4.14 (Pin_14)
- net lcd_db7: now also U?.14 (DB7)
- net lcd_rs: now reaches J4.15 (Pin_15)
- net lcd_rs: now also U?.4 (RS)
- net lcd_db6: now reaches J4.16 (Pin_16)
- net lcd_db6: now also U?.13 (DB6)
- net lcd_e: now reaches J4.24 (Pin_24)
- net lcd_e: now also U?.6 (E)
- net lcd_db5: now reaches J4.26 (Pin_26)
- net lcd_db5: now also U?.12 (DB5)
- net button: now reaches J4.5 (Pin_5)
- net at RV1.2: now also U?.3 (VO)
Other:
- moved on the sheet: RV1
Changed lines of the file:
@@
 $EndComp
 $Comp
-L k_digital_mix:P82B715 D1
+L mainboard-rescue:P82B715-k_digital_mix D1
 U 1 1 5DBDFBB1
 P 11850 1850
@@
 Text Notes 9000 3700 0    50   ~ 0
 НАДО ЛИ ДЕРГАТЬ ПИТАНИЕ I@C?
-$Comp
-L Connector_Generic:Conn_01x16 J1
-U 1 1 5DC8A30F
-P 5400 5500
-F 0 "J1" V 5524 5446 50  0000 C CNN
-F 1 "DISPLAY" V 5615 5446 50  0000 C CNN
-F 2 "Connector_PinHeader_2.54mm:PinHeader_1x16_P2.54mm_Vertical" H 5400 5500 50  0001 C CNN
-F 3 "~" H 5400 5500 50  0001 C CNN
-	1    5400 5500
-	0    -1   1    0
-$EndComp
 Wire Notes Line
 	3850 1600 7200 1600
@@
 Wire Notes Line
 	3850 4000 3850 1600
-Wire Notes Line
-	4500 5500 6900 5500
-Wire Notes Line
-	6900 5500 6900 6600
-Wire Notes Line
-	6900 6600 4500 6600
-Wire Notes Line
-	4500 6600 4500 5500
-Wire Notes Line
-	4700 5800 4700 6400
-Wire Notes Line
-	4700 6400 6700 6400
-Wire Notes Line
-	6700 6400 6700 5800
-Wire Notes Line
-	6700 5800 4700 5800
 $Comp
 L Device:R_POT RV1
 U 1 1 5DCA0042
-P 4900 4850
-F 0 "RV1" V 4693 4850 50  0000 C CNN
-F 1 "R_POT" V 4784 4850 50  0000 C CNN
-F 2 "" H 4900 4850 50  0001 C CNN
-F 3 "~" H 4900 4850 50  0001 C CNN
-	1    4900 4850
-	0    1    1    0
-$EndComp
-Wire Wire Line
-	4900 5000 4900 5300
-Wire Wire Line
-	5050 4850 5100 4850
-Wire Wire Line
-	5100 4850 5100 4950
-$Comp
-L power:GND #PWR0132
-U 1 1 5DCB151A
-P 5100 4950
-F 0 "#PWR0132" H 5100 4700 50  0001 C CNN
-F 1 "GND" H 5105 4777 50  0000 C CNN
-F 2 "" H 5100 4950 50  0001 C CNN
-F 3 "" H 5100 4950 50  0001 C CNN
-	1    5100 4950
-	1    0    0    -1
-$EndComp
-Wire Wire Line
-	4750 4850 4750 5100
-Wire Wire Line
-	4750 5100 4800 5100
-Wire Wire Line
-	4800 5100 4800 5300
-$Comp
-L power:GND #PWR0133
-U 1 1 5DCB5EFD
-P 4500 5250
-F 0 "#PWR0133" H 4500 5000 50  0001 C CNN
-F 1 "GND" H 4505 5077 50  0000 C CNN
-F 2 "" H 4500 5250 50  0001 C CNN
-F 3 "" H 4500 5250 50  0001 C CNN
-	1    4500 5250
-	1    0    0    -1
-$EndComp
-Wire Wire Line
-	4700 5300 4700 5200
-Wire Wire Line
-	4700 5200 4500 5200
-Wire Wire Line
-	4500 5200 4500 5250
-Wire Wire Line
-	6550 2800 5700 2800
-Wire Wire Line
-	5700 2800 5700 5300
-Wire Wire Line
-	5900 5300 5900 3000
-Wire Wire Line
-	5900 3000 6550 3000
-Wire Wire Line
-	7050 3000 7350 3000
-Wire Wire Line
-	7350 3000 7350 4500
-Wire Wire Line
-	7350 4500 6000 4500
-Wire Wire Line
-	6000 4500 6000 5300
-Wire Wire Line
-	7050 2900 7450 2900
-Wire Wire Line
-	7450 2900 7450 4600
-Wire Wire Line
-	7450 4600 5800 4600
-Wire Wire Line
-	5800 4600 5800 5300
+P 5400 4800
+F 0 "RV1" V 5193 4800 50  0000 C CNN
+F 1 "R_POT" V 5284 4800 50  0000 C CNN
+F 2 "" H 5400 4800 50  0001 C CNN
+F 3 "~" H 5400 4800 50  0001 C CNN
+	1    5400 4800
+	1    0    0    -1
+$EndComp
 Wire Wire Line
 	7050 2400 9600 2400
@@
 Wire Wire Line
 	7300 2100 7300 2150
+$Comp
+L Display_Character:LCD-016N002L U?
+U 1 1 5DCD6780
+P 5950 5400
+F 0 "U?" H 5950 6378 50  0000 C CNN
+F 1 "LCD-016N002L" H 5950 6287 50  0000 C CNN
+F 2 "Display:LCD-016N002L" H 5970 4480 50  0001 C CNN
+F 3 "http://www.vishay.com/docs/37299/37299.pdf" H 6450 5100 50  0001 C CNN
+	1    5950 5400
+	-1   0    0    -1
+$EndComp
+$Comp
+L power:+5V #PWR?
+U 1 1 5DD23078
+P 5400 4650
+F 0 "#PWR?" H 5400 4500 50  0001 C CNN
+F 1 "+5V" H 5415 4823 50  0000 C CNN
+F 2 "" H 5400 4650 50  0001 C CNN
+F 3 "" H 5400 4650 50  0001 C CNN
+	1    5400 4650
+	1    0    0    -1
+$EndComp
+$Comp
+L power:GND #PWR?
+U 1 1 5DD2319C
+P 5400 4950
+F 0 "#PWR?" H 5400 4700 50  0001 C CNN
+F 1 "GND" H 5405 4777 50  0000 C CNN
+F 2 "" H 5400 4950 50  0001 C CNN
+F 3 "" H 5400 4950 50  0001 C CNN
+	1    5400 4950
+	1    0    0    -1
+$EndComp
+$Comp
+L power:+5V #PWR?
+U 1 1 5DD9162C
+P 5950 4600
+F 0 "#PWR?" H 5950 4450 50  0001 C CNN
+F 1 "+5V" H 5965 4773 50  0000 C CNN
+F 2 "" H 5950 4600 50  0001 C CNN
+F 3 "" H 5950 4600 50  0001 C CNN
+	1    5950 4600
+	1    0    0    -1
+$EndComp
+$Comp
+L power:GND #PWR?
+U 1 1 5DD9182F
+P 5950 6200
+F 0 "#PWR?" H 5950 5950 50  0001 C CNN
+F 1 "GND" H 5955 6027 50  0000 C CNN
+F 2 "" H 5950 6200 50  0001 C CNN
+F 3 "" H 5950 6200 50  0001 C CNN
+	1    5950 6200
+	1    0    0    -1
+$EndComp
+$Comp
+L power:GND #PWR?
+U 1 1 5DDFEB95
+P 5550 5200
+F 0 "#PWR?" H 5550 4950 50  0001 C CNN
+F 1 "GND" H 5555 5027 50  0000 C CNN
+F 2 "" H 5550 5200 50  0001 C CNN
+F 3 "" H 5550 5200 50  0001 C CNN
+	1    5550 5200
+	1    0    0    -1
+$EndComp
+$Comp
+L power:+5V #PWR?
+U 1 1 5DDFECD8
+P 5550 5100
+F 0 "#PWR?" H 5550 4950 50  0001 C CNN
+F 1 "+5V" H 5565 5273 50  0000 C CNN
+F 2 "" H 5550 5100 50  0001 C CNN
+F 3 "" H 5550 5100 50  0001 C CNN
+	1    5550 5100
+	1    0    0    -1
+$EndComp
+Text Label 6350 5700 0    50   ~ 0
+lcd_db4
+Text Label 6350 5800 0    50   ~ 0
+lcd_db5
+Text Label 6350 5900 0    50   ~ 0
+lcd_db6
+Text Label 6350 6000 0    50   ~ 0
+lcd_db7
+Text Label 6350 4800 0    50   ~ 0
+lcd_e
+Text Label 6350 5000 0    50   ~ 0
+lcd_rs
+$Comp
+L power:GND #PWR?
+U 1 1 5DE091C2
+P 6350 4900
+F 0 "#PWR?" H 6350 4650 50  0001 C CNN
+F 1 "GND" V 6355 4772 50  0000 R CNN
+F 2 "" H 6350 4900 50  0001 C CNN
+F 3 "" H 6350 4900 50  0001 C CNN
+	1    6350 4900
+	0    -1   -1   0
+$EndComp
+Text Label 6550 3000 2    50   ~ 0
+lcd_rs
+Text Label 7050 3400 0    50   ~ 0
+lcd_e
+Text Label 7050 3500 0    50   ~ 0
+lcd_db5
+Text Label 7050 3000 0    50   ~ 0
+lcd_db6
+Text Label 7050 2900 0    50   ~ 0
+lcd_db7
+Text Label 6550 2900 2    50   ~ 0
+heat_24V
+Text Label 7050 2800 0    50   ~ 0
+i2c_rst
+Text Label 12850 3700 2    50   ~ 0
+i2c_rst
+Text Label 7050 2500 0    50   ~ 0
+valve1_12V
+Text Label 6550 2600 2    50   ~ 0
+valve2_12V
+Text Label 6550 2800 2    50   ~ 0
+lcd_db4
+Text Label 7050 2600 0    50   ~ 0
+valve3_12V
+Text Label 6550 2700 2    50   ~ 0
+valve4_12V
+Text Label 7050 2700 0    50   ~ 0
+valve5_12V
+Text Label 6550 2500 2    50   ~ 0
+button
+Text Label 6550 3200 2    50   ~ 0
+pump_24V
+Text Label 7050 3200 0    50   ~ 0
+fan_12V
+Text Label 6550 3300 2    50   ~ 0
+reserv_24V
 $EndSCHEMATC

Commit message: mainboard finished
Parts:
- removed J?: USB_A, symbol Connector:USB_A
- added C15: 0,1, Capacitor_SMD:C_0805_2012Metric_Pad1.15x1.40mm_HandSolder, symbol Device:C
- added J12: Conn_01x05, Connector_PinHeader_2.54mm:PinHeader_1x05_P2.54mm_Vertical, symbol Connector_Generic:Conn_01x05
- added J13: EXT3out, Connector_PinHeader_2.54mm:PinHeader_1x16_P2.54mm_Vertical, symbol Connector_Generic:Conn_01x16
- added J14, J15: Conn_01x01, Connector_Wire:SolderWirePad_1x01_Drill2mm, symbol Connector_Generic:Conn_01x01
- added J16: Conn_01x04, Connector_PinHeader_2.54mm:PinHeader_1x04_P2.54mm_Vertical, symbol Connector_Generic:Conn_01x04
- D1: symbol mainboard-rescue:P82B715-k_digital_mix -> k_digital_mix:P82B715
- J1: renamed from J?; footprint (none) -> Connector_IDC:IDC-Header_2x05_P2.54mm_Vertical
- RV1: footprint (none) -> Potentiometer_THT:Potentiometer_Bourns_3296W_Vertical
- U2: renamed from U?; footprint Display:LCD-016N002L -> Connector_PinHeader_2.54mm:PinHeader_1x16_P2.54mm_Vertical
- gave numbers to parts that had none: 5
Connections:
- net +3V3: now also J13.2 (Pin_2), J16.4 (Pin_4)
- net +5V: now also C15.2, J13.1 (Pin_1), J14.1 (Pin_1)
- net GND: now also C15.1, J13.16 (Pin_16), J15.1 (Pin_1), J16.1 (Pin_1)
- net at J2.25 (Pin_25): now also J12.4 (Pin_4)
- net at J2.3 (Pin_3): now also J12.5 (Pin_5)
- net at J4.17 (Pin_17): now also J12.3 (Pin_3)
- net at J4.18 (Pin_18): now also J12.1 (Pin_1)
- net at J4.22 (Pin_22): now also J12.2 (Pin_2)
- net at J4.23 (Pin_23): now also J16.3 (Pin_3)
- net at J4.25 (Pin_25): now also J16.2 (Pin_2)
- net at J3.10 (Pin_10): now also J13.10 (Pin_10)
- net at J3.11 (Pin_11): now also J13.11 (Pin_11)
- net at J3.12 (Pin_12): now also J13.12 (Pin_12)
- net at J3.13 (Pin_13): now also J13.13 (Pin_13)
- net at J3.14 (Pin_14): now also J13.14 (Pin_14)
- net at J3.15 (Pin_15): now also J13.15 (Pin_15)
- net at J3.3 (Pin_3): now also J13.3 (Pin_3)
- net at J3.4 (Pin_4): now also J13.4 (Pin_4)
- net at J3.5 (Pin_5): now also J13.5 (Pin_5)
- net at J3.6 (Pin_6): now also J13.6 (Pin_6)
- net at J3.7 (Pin_7): now also J13.7 (Pin_7)
- net at J3.8 (Pin_8): now also J13.8 (Pin_8)
- net at J3.9 (Pin_9): now also J13.9 (Pin_9)
Other:
- moved on the sheet: C11, C13, C14, J1, RV1, U2
