File: current_sensors/current_sensors.kicad_pcb (KiCad board)
At the start: 2 copper layers, 120 parts, among them J1 Conn_01x01, J10 Conn_02x05_Odd_Even, J11 Conn_01x01, J12 Conn_01x01, J13 Conn_01x01, J14 Conn_01x01, J15 Conn_01x01, J16 Conn_01x01, J17 Conn_01x01, J18 Conn_01x01, J19 Conn_01x01, J2 Conn_01x01, J20 Conn_01x01, J3 Conn_01x01, J4 Conn_01x01, J5 Conn_01x01, J6 Conn_01x01, J7 Conn_01x01, J8 Conn_01x01, J9 Conn_02x05_Odd_Even, U1 ACS758xCB-050B-PFF, U10 ACS712xLCTR-05B, U11 ACS712xLCTR-05B, U12 ACS712xLCTR-05B, U2 ACS758xCB-050B-PFF, U3 ACS712xLCTR-05B, U4 ACS712xLCTR-05B, U5 TL074, U6 TL074, U7 LM2901, U8 LM2901, U9 ACS712xLCTR-05B

Commit message: current-sensors: work in progress
Parts:
- J9: moved to B.Cu
- moved R15 240.6 mm to (56.5, 159.5), turned to 180 degrees
- moved C17 238.7 mm to (56.5, 127.0), turned to 180 degrees
- moved R3 236.9 mm to (56.5, 102.0), turned to 180 degrees
- moved C24 233.9 mm to (56.5, 177.0)
- moved R14 233.7 mm to (56.5, 144.5), turned to 180 degrees
- moved C21 233.5 mm to (56.5, 132.0)
- moved C10 228.8 mm to (67.5, 124.0), turned to 180 degrees
- moved C18 226.0 mm to (56.5, 142.0), turned to 180 degrees
- moved C2 224.4 mm to (75.0, 61.0), turned to 270 degrees
- moved C11 223.2 mm to (73.0, 124.0), turned to 180 degrees
- moved R13 222.8 mm to (56.5, 129.5), turned to 180 degrees
- moved C28 222.6 mm to (72.5, 159.0), turned to 180 degrees
- moved C22 222.2 mm to (56.5, 147.0)
- moved C26 220.2 mm to (67.0, 141.5), turned to 180 degrees
- moved R4 219.9 mm to (56.5, 114.5), turned to 180 degrees
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Connections:
- C14 pad 1: Net-(C14-Pad1) -> GND
- RV2 pad 3: Net-(C14-Pad1) -> GND
- U5 pad 1: Net-(C8-Pad1) -> Net-(C9-Pad1)
- U5 pad 13: Net-(C26-Pad2) -> Net-(C8-Pad2)
- U5 pad 14: Net-(C26-Pad1) -> Net-(C8-Pad1)
- U5 pad 2: Net-(C8-Pad2) -> Net-(C9-Pad2)
- U5 pad 6: Net-(C9-Pad2) -> Net-(C10-Pad2)
- U5 pad 7: Net-(C9-Pad1) -> Net-(C10-Pad1)
- U5 pad 8: Net-(C25-Pad1) -> Net-(C11-Pad1)
- U5 pad 9: Net-(C25-Pad2) -> Net-(C11-Pad2)
- U6 pad 1: Net-(C10-Pad1) -> Net-(C26-Pad1)
- U6 pad 13: Net-(C28-Pad2) -> Net-(C25-Pad2)
- U6 pad 14: Net-(C28-Pad1) -> Net-(C25-Pad1)
- U6 pad 2: Net-(C10-Pad2) -> Net-(C26-Pad2)
- U6 pad 6: Net-(C11-Pad2) -> Net-(C27-Pad2)
- U6 pad 7: Net-(C11-Pad1) -> Net-(C27-Pad1)
- U6 pad 8: Net-(C27-Pad1) -> Net-(C28-Pad1)
- U6 pad 9: Net-(C27-Pad2) -> Net-(C28-Pad2)

Commit message: current-sensors finished
Parts:
- added REF**: MountingHole_3.2mm_M3_Pad, MountingHole:MountingHole_3.2mm_M3_Pad, F.Cu at (135.0, 25.0)
- added REF**: MountingHole_3.2mm_M3_Pad, MountingHole:MountingHole_3.2mm_M3_Pad, F.Cu at (25.0, 25.0)
- added REF**: MountingHole_3.2mm_M3_Pad, MountingHole:MountingHole_3.2mm_M3_Pad, F.Cu at (135.0, 90.0)
- added REF**: MountingHole_3.2mm_M3_Pad, MountingHole:MountingHole_3.2mm_M3_Pad, F.Cu at (135.0, 155.0)
- added REF**: MountingHole_3.2mm_M3_Pad, MountingHole:MountingHole_3.2mm_M3_Pad, F.Cu at (25.0, 155.0)
- added REF**: MountingHole_3.2mm_M3_Pad, MountingHole:MountingHole_3.2mm_M3_Pad, F.Cu at (25.0, 90.0)
- D1, D2, D3, D4, D5, D6, D7, D8, F1, F2, F3, F4, F5, F6, F7, F8: moved to B.Cu
- J9: moved to F.Cu
- moved C35 129.5 mm to (99.0, 30.0), turned to 180 degrees
- moved J20 112.1 mm to (103.0, 25.0)
- moved J19 88.1 mm to (96.0, 25.0)
- moved C12 85.7 mm to (122.0, 39.0), turned to 270 degrees
- moved C36 76.6 mm to (97.5, 103.0)
- moved D2 74.6 mm to (125.0, 60.0), turned to 180 degrees
- moved R11 70.8 mm to (114.5, 95.0), turned to 90 degrees
- moved C1 69.9 mm to (76.8, 31.0), turned to 90 degrees
- moved D1 68.3 mm to (125.0, 45.0), turned to 180 degrees
- moved C31 68.3 mm to (111.0, 138.0), turned to 90 degrees
- moved C13 67.8 mm to (107.5, 83.0), turned to 270 degrees
- moved R9 67.5 mm to (117.5, 83.0), turned to 270 degrees
- moved D8 64.7 mm to (125.0, 150.0), turned to 180 degrees
- moved R10 64.6 mm to (115.0, 83.0), turned to 270 degrees
- moved C16 62.9 mm to (108.0, 95.0), turned to 90 degrees
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Connections:
- U7 pad 1: /Curr_2 -> /Curr_1
- U7 pad 10: Net-(C25-Pad1) -> Net-(C10-Pad1)
- U7 pad 11: Net-(C29-Pad2) -> Net-(C15-Pad2)
- U7 pad 13: /Curr_5 -> /Curr_3
- U7 pad 14: /Curr_6 -> /Curr_4
- U7 pad 2: /Curr_1 -> /Curr_2
- U7 pad 4: Net-(C8-Pad1) -> Net-(C9-Pad1)
- U7 pad 5: Net-(C13-Pad2) -> Net-(C14-Pad2)
- U7 pad 6: Net-(C9-Pad1) -> Net-(C8-Pad1)
- U7 pad 7: Net-(C14-Pad2) -> Net-(C13-Pad2)
- U7 pad 8: Net-(C26-Pad1) -> Net-(C11-Pad1)
- U7 pad 9: Net-(C30-Pad2) -> Net-(C16-Pad2)
- U8 pad 1: /Curr_4 -> /Curr_5
- U8 pad 2: /Curr_3 -> /Curr_6
- U8 pad 4: Net-(C10-Pad1) -> Net-(C26-Pad1)
- U8 pad 5: Net-(C15-Pad2) -> Net-(C30-Pad2)
- U8 pad 6: Net-(C11-Pad1) -> Net-(C25-Pad1)
- U8 pad 7: Net-(C16-Pad2) -> Net-(C29-Pad2)
Routing:
- net GND: track 0.00 -> 692.1 mm, vias 0 -> 26
- net +5V: track 0.00 -> 501.6 mm, vias 0 -> 2
- net /Curr_8: track 0.00 -> 197.4 mm
- net /Volt_8: track 0.00 -> 182.3 mm, vias 0 -> 1
- net /Curr_7: track 0.00 -> 172.0 mm
- net /Volt_4: track 0.00 -> 168.7 mm
- net /Volt_7: track 0.00 -> 167.1 mm, vias 0 -> 1
- net /Curr_6: track 0.00 -> 156.9 mm
- net /Volt_6: track 0.00 -> 151.4 mm, vias 0 -> 1
- net /Volt_3: track 0.00 -> 150.7 mm
- net /Curr_5: track 0.00 -> 136.9 mm
- net /Volt_5: track 0.00 -> 135.6 mm, vias 0 -> 1
- net /Volt_2: track 0.00 -> 132.2 mm
- net /Volt_1: track 0.00 -> 103.7 mm
- net /Curr_4: track 0.00 -> 95.0 mm
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Other:
- board outline added: 120 x 140 mm
- net class Default: trace_width 0.25 -> 0.3
