File: current_sensors/current_sensors.sch (KiCad schematic (older format))
At the start: 49 parts, among them J1 Conn_01x01, J10 Conn_01x01, J11 Conn_01x01, J12 Conn_01x01, J13 Conn_01x01, J14 Conn_01x01, J15 Conn_02x05_Odd_Even, J16 Conn_01x01, J17 Conn_01x01, J18 Conn_01x05, J2 Conn_01x01, J3 Conn_01x01, J4 Conn_01x01, J5 Conn_01x01, J6 Conn_01x01, J7 Conn_01x01, J8 Conn_01x01, J9 Conn_01x01, U1 ACS758xCB-050B-PFF, U2 ACS758xCB-050B-PFF, U3 ACS712xLCTR-05B

Commit message: current sensors: work in progress
Parts:
- removed F2: Fuse, symbol Device:Fuse
- removed J10, J11, J12, J3, J4, J9: Conn_01x01, symbol Connector_Generic:Conn_01x01
- removed J15: Conn_02x05_Odd_Even, symbol Connector_Generic:Conn_02x05_Odd_Even
- removed J18: Conn_01x05, symbol Connector_Generic:Conn_01x05
- removed U2: ACS758xCB-050B-PFF, Sensor_Current:Allegro_CB_PFF, symbol Sensor_Current:ACS758xCB-050B-PFF
- added C1, C12, C13, C15, C16, C18, C19, C20, C30, C31, C32, C33, C34, C35, C37, C38, C4, C5: 0,1, symbol Device:C
- added C10, C11, C26, C27, C28, C8: C*, symbol Device:C
- added C22, C23, C24, C6, C7: C, symbol Device:C
- added D1, D3, D4, D6, D7, D8: LED, symbol Device:LED
- added F1, F3, F4, F6, F7, F8: Fuse, symbol Device:Fuse
- added J1, J15, J16, J17, J18, J19, J2, J20: Conn_01x01, symbol Connector_Generic:Conn_01x01
- added J10, J9: Conn_02x05_Odd_Even, symbol Connector_Generic:Conn_02x05_Odd_Even
- added R1, R14, R15, R16, R3, R4: 7,5k, symbol Device:R
- added R11, R12, R22, R23, R24, R9: *, symbol Device:R
- added R18, R19, R20, R5, R7, R8: 30k, symbol Device:R
- added RV1, RV3, RV4, RV6, RV7, RV8: R_POT, symbol Device:R_POT
- added U1: ACS758xCB-050B-PFF, Sensor_Current:Allegro_CB_PFF, symbol Sensor_Current:ACS758xCB-050B-PFF
- added U10, U11, U12, U3, U4: ACS712xLCTR-05B, Package_SO:SOIC-8_3.9x4.9mm_P1.27mm, symbol Sensor_Current:ACS712xLCTR-05B
- added unit 1 of U5
- added unit 4 of U5
- added unit 5 of U5
- added U6: TL074, symbol Amplifier_Operational:TL074
- added unit 1 of U7
- added unit 4 of U7
- added unit 5 of U7
- added U8: LM2901, symbol Comparator:LM2901
- gave numbers to parts that had none: 19
- renumbered C3 to C17, C4 to C21, C1 to C3, F1 to F2, F3 to F5, J16 to J11, J17 to J12, J1 to J3, J2 to J4, U1 to U2, U3 to U9
Connections:
- net +5V: now also C1.1, C12.1, C18.2, C19.2, C20.2, C33.2, C34.2, C35.2, C37.2, C38.2, C4.2, C5.2, J10.2 (Pin_2), J19.1 (Pin_1), J9.2 (Pin_2), R11.1, R12.1, R22.1, R23.1, R24.1, R9.1, RV1.1, RV3.1, RV4.1, RV6.1, RV7.1, RV8.1, U1.1 (VCC), U10.8 (VCC), U11.8 (VCC), U12.8 (VCC), U3.8 (VCC), U4.8 (VCC), U5.4 (V+), U6.4 (V+), U7.3 (V+), U8.3 (V+)
- net GND: now also C1.2, C12.2, C13.1, C15.1, C16.1, C18.1, C19.1, C20.1, C22.2, C23.2, C24.2, C30.1, C31.1, C32.1, C33.1, C34.1, C35.1, C37.1, C38.1, C4.1, C5.1, C6.2, C7.2, D1.1 (K), D3.1 (K), D4.1 (K), D6.1 (K), D7.1 (K), D8.1 (K), J10.1 (Pin_1), J20.1 (Pin_1), J9.1 (Pin_1), RV1.3, RV3.3, RV4.3, RV6.3, RV7.3, RV8.3, U1.2 (GND), U10.5 (GND), U11.5 (GND), U12.5 (GND), U3.5 (GND), U4.5 (GND), U5.11 (V-), U6.11 (V-), U7.12 (V-), U8.12 (V-); no longer C14.1, RV2.3
- net Vcc\2: now also U5.10 (+), U5.5 (+), U5.12 (+), U5.3 (+), U6.10 (+), U6.12 (+), U6.3 (+), U6.5 (+); no longer U5.3 (+), U5.3 (+)
- net Volt_5: now reaches J12.1 (Pin_1), U9.3 (IP-), U9.4 (IP-)
- net Volt_5: now also J9.10 (Pin_10)
- net at U2.3 (VIOUT): now also R2.2
- net Volt_2: now reaches J4.1 (Pin_1), U2.5 (IP-)
- net Volt_2: now also J9.5 (Pin_5)
- net at C25.1, R17.1: now also U5.8, U7.10 (-); no longer U5.1, U7.4 (-)
- net at C25.2, R13.1, R17.2: now also U5.9 (-); no longer U5.2 (-)
- net Curr_5: now reaches D5.2 (A), R21.2
- net Curr_5: now also U7.13, J10.10 (Pin_10); no longer U7.2
- net at C29.2, RV5.2: now also U7.11 (+); no longer U7.5 (+)
- net at C9.1, R6.1: now also U5.7, U7.6 (-); no longer U5.1, U7.4 (-)
- net at C9.2, R2.1, R6.2: now also U5.6 (-); no longer U5.2 (-)
- net Curr_2: now reaches D2.2 (A), R10.2
- net Curr_2: now also U7.1, J10.5 (Pin_5); no longer U7.2
- net at C14.2, RV2.2: now also U7.7 (+); no longer U7.5 (+)
- removed net +12VA: J13.1 (Pin_1), J14.1 (Pin_1), J5.1 (Pin_1), J6.1 (Pin_1), J7.1 (Pin_1), J8.1 (Pin_1)
- new net: C14.1, RV2.3
- new net: R1.2, U1.3 (VIOUT)
- new net: F1.1, U1.4 (IP+)
- new net: F1.2, J1.1 (Pin_1)
- new net: C8.1, R5.1, U5.1, U7.4 (-)
- new net: C8.2, R1.1, R5.2, U5.2 (-)
- new net: C13.2, RV1.2, U7.5 (+)
- new net: F6.1, U10.1 (IP+), U10.2 (IP+)
- new net: C22.1, U10.6 (FILTER)
- new net: R14.2, U10.7 (VIOUT)
- new net: F6.2, J13.1 (Pin_1)
- new net: C26.2, R14.1, R18.2, U5.13 (-)
- new net: C26.1, R18.1, U5.14, U7.8 (-)
- new net: C30.2, RV6.2, U7.9 (+)
- new net: F3.1, U3.1 (IP+), U3.2 (IP+)
- new net: C6.1, U3.6 (FILTER)
- new net: R3.2, U3.7 (VIOUT)
- new net: F3.2, J5.1 (Pin_1)
- new net: C10.1, R7.1, U6.1, U8.4 (-)
- new net: C10.2, R3.1, R7.2, U6.2 (-)
- new net: C15.2, RV3.2, U8.5 (+)
- new net: F4.1, U4.1 (IP+), U4.2 (IP+)
- new net: C7.1, U4.6 (FILTER)
- new net: R4.2, U4.7 (VIOUT)
- new net: F4.2, J7.1 (Pin_1)
- new net: C11.2, R4.1, R8.2, U6.6 (-)
- new net: C11.1, R8.1, U6.7, U8.6 (-)
- new net: C16.2, RV4.2, U8.7 (+)
- new net: F7.1, U11.1 (IP+), U11.2 (IP+)
- new net: C23.1, U11.6 (FILTER)
- new net: R15.2, U11.7 (VIOUT)
- new net: F7.2, J15.1 (Pin_1)
- new net: C27.1, R19.1, U6.8, U8.10 (-)
- new net: C27.2, R15.1, R19.2, U6.9 (-)
- new net: C31.2, RV7.2, U8.11 (+)
- new net: F8.1, U12.1 (IP+), U12.2 (IP+)
- new net: C24.1, U12.6 (FILTER)
- new net: R16.2, U12.7 (VIOUT)
- new net: F8.2, J17.1 (Pin_1)
- new net: C28.2, R16.1, R20.2, U6.13 (-)
- new net: C28.1, R20.1, U6.14, U8.8 (-)
- new net: C32.2, RV8.2, U8.9 (+)
- new net Curr_1: D1.2 (A), J10.3 (Pin_3), R9.2, U7.2
- new net Curr_3: D3.2 (A), J10.7 (Pin_7), R11.2, U8.2
- new net Curr_4: D4.2 (A), J10.9 (Pin_9), R12.2, U8.1
- new net Curr_6: D6.2 (A), J10.8 (Pin_8), R22.2, U7.14
- new net Curr_7: D7.2 (A), J10.6 (Pin_6), R23.2, U8.13
- new net Curr_8: D8.2 (A), J10.4 (Pin_4), R24.2, U8.14
- new net Volt_1: J2.1 (Pin_1), J9.3 (Pin_3), U1.5 (IP-)
- new net Volt_3: J6.1 (Pin_1), J9.7 (Pin_7), U3.3 (IP-), U3.4 (IP-)
- new net Volt_4: J8.1 (Pin_1), J9.9 (Pin_9), U4.3 (IP-), U4.4 (IP-)
- new net Volt_6: J14.1 (Pin_1), J9.8 (Pin_8), U10.3 (IP-), U10.4 (IP-)
- new net Volt_7: J16.1 (Pin_1), J9.6 (Pin_6), U11.3 (IP-), U11.4 (IP-)
- new net Volt_8: J18.1 (Pin_1), J9.4 (Pin_4), U12.3 (IP-), U12.4 (IP-)
Other:
- moved on the sheet: C14, C17, C21, C25, C29, C3, C36, C9, D2, D5, F2, F5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

Commit message: HTU bufer added
Parts:
- C1, C10, C11, C12, C13, C14, C15, C16, C17, C18, C19, C2, C20, C21, C22, C23, C24, C25, C26, C27, C28, C29, C3, C30, C31, C32, C33, C34, C35, C36, C37, C38, C4, C5, C6, C7, C8, C9: footprint (none) -> Capacitor_SMD:C_0805_2012Metric_Pad1.15x1.40mm_HandSolder
- D1, D2, D3, D4, D5, D6, D7, D8: footprint (none) -> LED_THT:LED_D5.0mm
- F1, F2, F3, F4, F5, F6, F7, F8: footprint (none) -> Fuse:Fuseholder_Cylinder-5x20mm_Schurter_0031_8201_Horizontal_Open
- J1, J11, J12, J13, J14, J15, J16, J17, J18, J19, J2, J20, J3, J4, J5, J6, J7, J8: footprint (none) -> Connector_Wire:SolderWirePad_1x01_Drill2mm
- J10, J9: footprint (none) -> Connector_IDC:IDC-Header_2x05_P2.54mm_Vertical
- R1, R10, R11, R12, R13, R14, R15, R16, R17, R18, R19, R2, R20, R21, R22, R23, R24, R25, R26, R3, R4, R5, R6, R7, R8, R9: footprint (none) -> Resistor_SMD:R_0805_2012Metric_Pad1.15x1.40mm_HandSolder
- RV1, RV2, RV3, RV4, RV5, RV6, RV7, RV8: footprint (none) -> Potentiometer_THT:Potentiometer_Bourns_3296W_Vertical
- U5, U6, U7, U8: footprint (none) -> Package_SO:SOIC-14_3.9x8.7mm_P1.27mm
Connections:
- net GND: now also C14.1, RV2.3

Commit message: current-sensors: work in progress
Connections:
- net at C25.1, R17.1, U7.10 (-): now also U6.14; no longer U5.8
- net at C25.2, R13.1, R17.2: now also U6.13 (-); no longer U5.9 (-)
- net at C9.2, R2.1, R6.2: now also U5.2 (-); no longer U5.6 (-)
- net at C9.1, R6.1, U7.6 (-): now also U5.1; no longer U5.7
- net at C8.1, R5.1, U7.4 (-): now also U5.14; no longer U5.1
- net at C8.2, R1.1, R5.2: now also U5.13 (-); no longer U5.2 (-)
- net at C26.2, R14.1, R18.2: now also U6.2 (-); no longer U5.13 (-)
- net at C26.1, R18.1, U7.8 (-): now also U6.1; no longer U5.14
- net at C10.1, R7.1, U8.4 (-): now also U5.7; no longer U6.1
- net at C10.2, R3.1, R7.2: now also U5.6 (-); no longer U6.2 (-)
- net at C11.2, R4.1, R8.2: now also U5.9 (-); no longer U6.6 (-)
- net at C11.1, R8.1, U8.6 (-): now also U5.8; no longer U6.7
- net at C27.1, R19.1, U8.10 (-): now also U6.7; no longer U6.8
- net at C27.2, R15.1, R19.2: now also U6.6 (-); no longer U6.9 (-)
- net at C28.2, R16.1, R20.2: now also U6.9 (-); no longer U6.13 (-)
- net at C28.1, R20.1, U8.8 (-): now also U6.8; no longer U6.14
Other:
- moved on the sheet: U5A, U5B, U5C, U5D, U6A, U6B, U6C, U6D
Changed lines of the file:
@@
 L Amplifier_Operational:TL074 U5
 U 3 1 5DC0304C
-P 9700 1800
-F 0 "U5" H 9700 2167 50  0000 C CNN
-F 1 "TL074" H 9700 2076 50  0000 C CNN
-F 2 "Package_SO:SOIC-14_3.9x8.7mm_P1.27mm" H 9650 1900 50  0001 C CNN
-F 3 "http://www.ti.com/lit/ds/symlink/tl071.pdf" H 9750 2000 50  0001 C CNN
-	3    9700 1800
+P 3650 7050
+F 0 "U5" H 3650 7417 50  0000 C CNN
+F 1 "TL074" H 3650 7326 50  0000 C CNN
+F 2 "Package_SO:SOIC-14_3.9x8.7mm_P1.27mm" H 3600 7150 50  0001 C CNN
+F 3 "http://www.ti.com/lit/ds/symlink/tl071.pdf" H 3700 7250 50  0001 C CNN
+	3    3650 7050
 	1    0    0    1
 $EndComp
@@
 L Amplifier_Operational:TL074 U5
 U 2 1 5DC36C1D
-P 3500 3300
-F 0 "U5" H 3500 3667 50  0000 C CNN
-F 1 "TL074" H 3500 3576 50  0000 C CNN
-F 2 "Package_SO:SOIC-14_3.9x8.7mm_P1.27mm" H 3450 3400 50  0001 C CNN
-F 3 "http://www.ti.com/lit/ds/symlink/tl071.pdf" H 3550 3500 50  0001 C CNN
-	2    3500 3300
+P 3650 5300
+F 0 "U5" H 3650 5667 50  0000 C CNN
+F 1 "TL074" H 3650 5576 50  0000 C CNN
+F 2 "Package_SO:SOIC-14_3.9x8.7mm_P1.27mm" H 3600 5400 50  0001 C CNN
+F 3 "http://www.ti.com/lit/ds/symlink/tl071.pdf" H 3700 5500 50  0001 C CNN
+	2    3650 5300
 	1    0    0    1
 $EndComp
@@
 L Amplifier_Operational:TL074 U5
 U 1 1 5DCF6CD2
-P 3500 1600
-F 0 "U5" H 3500 1967 50  0000 C CNN
-F 1 "TL074" H 3500 1876 50  0000 C CNN
-F 2 "Package_SO:SOIC-14_3.9x8.7mm_P1.27mm" H 3450 1700 50  0001 C CNN
-F 3 "http://www.ti.com/lit/ds/symlink/tl071.pdf" H 3550 1800 50  0001 C CNN
-	1    3500 1600
+P 3500 3300
+F 0 "U5" H 3500 3667 50  0000 C CNN
+F 1 "TL074" H 3500 3576 50  0000 C CNN
+F 2 "Package_SO:SOIC-14_3.9x8.7mm_P1.27mm" H 3450 3400 50  0001 C CNN
+F 3 "http://www.ti.com/lit/ds/symlink/tl071.pdf" H 3550 3500 50  0001 C CNN
+	1    3500 3300
 	1    0    0    1
 $EndComp
@@
 L Amplifier_Operational:TL074 U5
 U 4 1 5DD05522
-P 9700 3550
-F 0 "U5" H 9700 3917 50  0000 C CNN
-F 1 "TL074" H 9700 3826 50  0000 C CNN
-F 2 "Package_SO:SOIC-14_3.9x8.7mm_P1.27mm" H 9650 3650 50  0001 C CNN
-F 3 "http://www.ti.com/lit/ds/symlink/tl071.pdf" H 9750 3750 50  0001 C CNN
-	4    9700 3550
+P 3500 1600
+F 0 "U5" H 3500 1967 50  0000 C CNN
+F 1 "TL074" H 3500 1876 50  0000 C CNN
+F 2 "Package_SO:SOIC-14_3.9x8.7mm_P1.27mm" H 3450 1700 50  0001 C CNN
+F 3 "http://www.ti.com/lit/ds/symlink/tl071.pdf" H 3550 1800 50  0001 C CNN
+	4    3500 1600
 	1    0    0    1
 $EndComp
@@
 L Amplifier_Operational:TL074 U6
 U 1 1 5DD0CB8C
-P 3650 5300
-F 0 "U6" H 3650 5667 50  0000 C CNN
-F 1 "TL074" H 3650 5576 50  0000 C CNN
-F 2 "Package_SO:SOIC-14_3.9x8.7mm_P1.27mm" H 3600 5400 50  0001 C CNN
-F 3 "http://www.ti.com/lit/ds/symlink/tl071.pdf" H 3700 5500 50  0001 C CNN
-	1    3650 5300
+P 9700 3550
+F 0 "U6" H 9700 3917 50  0000 C CNN
+F 1 "TL074" H 9700 3826 50  0000 C CNN
+F 2 "Package_SO:SOIC-14_3.9x8.7mm_P1.27mm" H 9650 3650 50  0001 C CNN
+F 3 "http://www.ti.com/lit/ds/symlink/tl071.pdf" H 9750 3750 50  0001 C CNN
+	1    9700 3550
 	1    0    0    1
 $EndComp
@@
 L Amplifier_Operational:TL074 U6
 U 2 1 5DD0CC4A
-P 3650 7050
-F 0 "U6" H 3650 7417 50  0000 C CNN
-F 1 "TL074" H 3650 7326 50  0000 C CNN
-F 2 "Package_SO:SOIC-14_3.9x8.7mm_P1.27mm" H 3600 7150 50  0001 C CNN
-F 3 "http://www.ti.com/lit/ds/symlink/tl071.pdf" H 3700 7250 50  0001 C CNN
-	2    3650 7050
+P 9700 5400
+F 0 "U6" H 9700 5767 50  0000 C CNN
+F 1 "TL074" H 9700 5676 50  0000 C CNN
+F 2 "Package_SO:SOIC-14_3.9x8.7mm_P1.27mm" H 9650 5500 50  0001 C CNN
+F 3 "http://www.ti.com/lit/ds/symlink/tl071.pdf" H 9750 5600 50  0001 C CNN
+	2    9700 5400
 	1    0    0    1
 $EndComp
@@
 L Amplifier_Operational:TL074 U6
 U 3 1 5DD1CAAB
-P 9700 5400
-F 0 "U6" H 9700 5767 50  0000 C CNN
-F 1 "TL074" H 9700 5676 50  0000 C CNN
-F 2 "Package_SO:SOIC-14_3.9x8.7mm_P1.27mm" H 9650 5500 50  0001 C CNN
-F 3 "http://www.ti.com/lit/ds/symlink/tl071.pdf" H 9750 5600 50  0001 C CNN
-	3    9700 5400
+P 9700 7150
+F 0 "U6" H 9700 7517 50  0000 C CNN
+F 1 "TL074" H 9700 7426 50  0000 C CNN
+F 2 "Package_SO:SOIC-14_3.9x8.7mm_P1.27mm" H 9650 7250 50  0001 C CNN
+F 3 "http://www.ti.com/lit/ds/symlink/tl071.pdf" H 9750 7350 50  0001 C CNN
+	3    9700 7150
 	1    0    0    1
 $EndComp
@@
 L Amplifier_Operational:TL074 U6
 U 4 1 5DD1CB69
-P 9700 7150
-F 0 "U6" H 9700 7517 50  0000 C CNN
-F 1 "TL074" H 9700 7426 50  0000 C CNN
-F 2 "Package_SO:SOIC-14_3.9x8.7mm_P1.27mm" H 9650 7250 50  0001 C CNN
-F 3 "http://www.ti.com/lit/ds/symlink/tl071.pdf" H 9750 7350 50  0001 C CNN
-	4    9700 7150
+P 9700 1800
+F 0 "U6" H 9700 2167 50  0000 C CNN
+F 1 "TL074" H 9700 2076 50  0000 C CNN
+F 2 "Package_SO:SOIC-14_3.9x8.7mm_P1.27mm" H 9650 1900 50  0001 C CNN
+F 3 "http://www.ti.com/lit/ds/symlink/tl071.pdf" H 9750 2000 50  0001 C CNN
+	4    9700 1800
 	1    0    0    1
 $EndComp

Commit message: current-sensors finished
Connections:
- net Curr_1: now also U7.1; no longer U7.2
- net Curr_2: now also U7.2; no longer U7.1
- net Curr_3: now also U7.13; no longer U8.2
- net Curr_4: now also U7.14; no longer U8.1
- net Curr_5: now also U8.1; no longer U7.13
- net Curr_6: now also U8.2; no longer U7.14
- net at C11.1, R8.1, U5.8: now also U7.8 (-); no longer U8.6 (-)
- net at C25.1, R17.1, U6.14: now also U8.6 (-); no longer U7.10 (-)
- net at C29.2, RV5.2: now also U8.7 (+); no longer U7.11 (+)
- net at C10.1, R7.1, U5.7: now also U7.10 (-); no longer U8.4 (-)
- net at C9.1, R6.1, U5.1: now also U7.4 (-); no longer U7.6 (-)
- net at C14.2, RV2.2: now also U7.5 (+); no longer U7.7 (+)
- net at C8.1, R5.1, U5.14: now also U7.6 (-); no longer U7.4 (-)
- net at C13.2, RV1.2: now also U7.7 (+); no longer U7.5 (+)
- net at C26.1, R18.1, U6.1: now also U8.4 (-); no longer U7.8 (-)
- net at C30.2, RV6.2: now also U8.5 (+); no longer U7.9 (+)
- net at C15.2, RV3.2: now also U7.11 (+); no longer U8.5 (+)
- net at C16.2, RV4.2: now also U7.9 (+); no longer U8.7 (+)
Other:
- moved on the sheet: U7A, U7B, U7C, U7D, U8A, U8B
Changed lines of the file:
@@
 L Comparator:LM2901 U7
 U 3 1 5DC108C9
-P 11100 1900
-F 0 "U7" H 11100 1533 50  0000 C CNN
-F 1 "LM2901" H 11100 1624 50  0000 C CNN
-F 2 "Package_SO:SOIC-14_3.9x8.7mm_P1.27mm" H 11050 2000 50  0001 C CNN
-F 3 "http://www.ti.com/lit/ds/symlink/lm339.pdf" H 11150 2100 50  0001 C CNN
-	3    11100 1900
+P 5050 5400
+F 0 "U7" H 5050 5033 50  0000 C CNN
+F 1 "LM2901" H 5050 5124 50  0000 C CNN
+F 2 "Package_SO:SOIC-14_3.9x8.7mm_P1.27mm" H 5000 5500 50  0001 C CNN
+F 3 "http://www.ti.com/lit/ds/symlink/lm339.pdf" H 5100 5600 50  0001 C CNN
+	3    5050 5400
 	1    0    0    1
 $EndComp
@@
 L Comparator:LM2901 U7
 U 2 1 5DC36C23
-P 4900 3400
-F 0 "U7" H 4900 3033 50  0000 C CNN
-F 1 "LM2901" H 4900 3124 50  0000 C CNN
-F 2 "Package_SO:SOIC-14_3.9x8.7mm_P1.27mm" H 4850 3500 50  0001 C CNN
-F 3 "http://www.ti.com/lit/ds/symlink/lm339.pdf" H 4950 3600 50  0001 C CNN
-	2    4900 3400
+P 4900 1700
+F 0 "U7" H 4900 1333 50  0000 C CNN
+F 1 "LM2901" H 4900 1424 50  0000 C CNN
+F 2 "Package_SO:SOIC-14_3.9x8.7mm_P1.27mm" H 4850 1800 50  0001 C CNN
+F 3 "http://www.ti.com/lit/ds/symlink/lm339.pdf" H 4950 1900 50  0001 C CNN
+	2    4900 1700
 	1    0    0    1
 $EndComp
@@
 L Comparator:LM2901 U7
 U 1 1 5DCF6CD8
-P 4900 1700
-F 0 "U7" H 4900 1333 50  0000 C CNN
-F 1 "LM2901" H 4900 1424 50  0000 C CNN
-F 2 "Package_SO:SOIC-14_3.9x8.7mm_P1.27mm" H 4850 1800 50  0001 C CNN
-F 3 "http://www.ti.com/lit/ds/symlink/lm339.pdf" H 4950 1900 50  0001 C CNN
-	1    4900 1700
+P 4900 3400
+F 0 "U7" H 4900 3033 50  0000 C CNN
+F 1 "LM2901" H 4900 3124 50  0000 C CNN
+F 2 "Package_SO:SOIC-14_3.9x8.7mm_P1.27mm" H 4850 3500 50  0001 C CNN
+F 3 "http://www.ti.com/lit/ds/symlink/lm339.pdf" H 4950 3600 50  0001 C CNN
+	1    4900 3400
 	1    0    0    1
 $EndComp
@@
 L Comparator:LM2901 U7
 U 4 1 5DD05528
-P 11100 3650
-F 0 "U7" H 11100 3283 50  0000 C CNN
-F 1 "LM2901" H 11100 3374 50  0000 C CNN
-F 2 "Package_SO:SOIC-14_3.9x8.7mm_P1.27mm" H 11050 3750 50  0001 C CNN
-F 3 "http://www.ti.com/lit/ds/symlink/lm339.pdf" H 11150 3850 50  0001 C CNN
-	4    11100 3650
+P 5050 7150
+F 0 "U7" H 5050 6783 50  0000 C CNN
+F 1 "LM2901" H 5050 6874 50  0000 C CNN
+F 2 "Package_SO:SOIC-14_3.9x8.7mm_P1.27mm" H 5000 7250 50  0001 C CNN
+F 3 "http://www.ti.com/lit/ds/symlink/lm339.pdf" H 5100 7350 50  0001 C CNN
+	4    5050 7150
 	1    0    0    1
 $EndComp
@@
 L Comparator:LM2901 U8
 U 1 1 5DD0CB92
-P 5050 5400
-F 0 "U8" H 5050 5033 50  0000 C CNN
-F 1 "LM2901" H 5050 5124 50  0000 C CNN
-F 2 "Package_SO:SOIC-14_3.9x8.7mm_P1.27mm" H 5000 5500 50  0001 C CNN
-F 3 "http://www.ti.com/lit/ds/symlink/lm339.pdf" H 5100 5600 50  0001 C CNN
-	1    5050 5400
+P 11100 3650
+F 0 "U8" H 11100 3283 50  0000 C CNN
+F 1 "LM2901" H 11100 3374 50  0000 C CNN
+F 2 "Package_SO:SOIC-14_3.9x8.7mm_P1.27mm" H 11050 3750 50  0001 C CNN
+F 3 "http://www.ti.com/lit/ds/symlink/lm339.pdf" H 11150 3850 50  0001 C CNN
+	1    11100 3650
 	1    0    0    1
 $EndComp
@@
 L Comparator:LM2901 U8
 U 2 1 5DD0CC50
-P 5050 7150
-F 0 "U8" H 5050 6783 50  0000 C CNN
-F 1 "LM2901" H 5050 6874 50  0000 C CNN
-F 2 "Package_SO:SOIC-14_3.9x8.7mm_P1.27mm" H 5000 7250 50  0001 C CNN
-F 3 "http://www.ti.com/lit/ds/symlink/lm339.pdf" H 5100 7350 50  0001 C CNN
-	2    5050 7150
+P 11100 1900
+F 0 "U8" H 11100 1533 50  0000 C CNN
+F 1 "LM2901" H 11100 1624 50  0000 C CNN
+F 2 "Package_SO:SOIC-14_3.9x8.7mm_P1.27mm" H 11050 2000 50  0001 C CNN
+F 3 "http://www.ti.com/lit/ds/symlink/lm339.pdf" H 11150 2100 50  0001 C CNN
+	2    11100 1900
 	1    0    0    1
 $EndComp
