File: 5V_supply/5V_supply.kicad_pcb (KiCad board)
At the start: 2 copper layers, 100 x 70 mm, 15 parts, among them J1 Conn_01x01, J2 Conn_01x01, J3 Conn_01x01, J4 Conn_01x01, J5 Conn_01x01, J6 Conn_01x01, J7 Conn_01x01, J8 Conn_01x01

Commit message: power supply finished
Parts:
- removed C1: 0,47x630V, Capacitor_THT:C_Rect_L33.0mm_W15.0mm_P27.50mm_MKS4
- removed C2: 0,1, Capacitor_THT:C_Rect_L7.0mm_W3.5mm_P5.00mm
- added F1: Fuse, Fuse:Fuseholder_Cylinder-5x20mm_Schurter_0031_8201_Horizontal_Open, F.Cu at (105.0, 50.0)
- added J10: Conn_01x01, Connector_Wire:SolderWirePad_1x01_Drill2.5mm, F.Cu at (130.0, 85.0)
- added J11: Conn_01x01, Connector_Wire:SolderWirePad_1x01_Drill2.5mm, F.Cu at (150.0, 65.0)
- added J12: Conn_01x01, Connector_Wire:SolderWirePad_1x01_Drill2.5mm, F.Cu at (150.0, 75.0)
- added J13: Conn_01x01, Connector_Wire:SolderWirePad_1x01_Drill2.5mm, F.Cu at (150.0, 85.0)
- added J9: Conn_01x01, Connector_Wire:SolderWirePad_1x01_Drill2.5mm, F.Cu at (130.0, 65.0)
- added REF**: MountingHole_3.2mm_M3_Pad, MountingHole:MountingHole_3.2mm_M3_Pad, F.Cu at (120.0, 102.5)
- added REF**: MountingHole_3.2mm_M3_Pad, MountingHole:MountingHole_3.2mm_M3_Pad, F.Cu at (120.0, 47.5)
- moved C3 34.9 mm to (145.0, 102.5), turned to 90 degrees
- moved J1 28.8 mm to (75.0, 55.0)
- moved J2 28.0 mm to (75.0, 92.5)
- moved REF** 25.1 mm to (160.0, 47.5)
- moved REF** 25.1 mm to (160.0, 102.5)
- moved J7 24.5 mm to (160.0, 65.0)
- moved J8 24.5 mm to (160.0, 85.0)
- moved REF** 10.3 mm to (40.0, 47.5)
- moved REF** 10.3 mm to (40.0, 102.5)
Connections:
- C3 pad 1: Net-(C2-Pad1) -> Net-(C3-Pad1)
- C3 pad 2: Net-(C2-Pad2) -> Net-(C3-Pad2)
- J1 pad 1: Net-(C1-Pad1) -> Net-(F1-Pad2)
- J3 pad 1: Net-(C1-Pad1) -> Net-(F1-Pad1)
- J5 pad 1: Net-(C2-Pad1) -> Net-(J5-Pad1)
- J6 pad 1: Net-(C2-Pad2) -> Net-(J10-Pad1)
- J7 pad 1: Net-(C2-Pad1) -> Net-(C3-Pad1)
- J8 pad 1: Net-(C2-Pad2) -> Net-(C3-Pad2)
Routing:
- net Net-(C3-Pad1): track 0.00 -> 122.4 mm
- net Net-(F1-Pad1): track 0.00 -> 77.6 mm
- net Net-(C2-Pad2): track 67.8 -> 0.00 mm
- net Net-(C1-Pad1): track 64.2 -> 0.00 mm
- net Net-(C2-Pad1): track 60.3 -> 0.00 mm
- net Net-(J2-Pad1): track 60.4 -> 16.0 mm
- net Net-(C3-Pad2): track 0.00 -> 44.1 mm
- net Net-(J5-Pad1): track 0.00 -> 38.6 mm
- net Net-(J10-Pad1): track 0.00 -> 20.4 mm
- net Net-(F1-Pad2): track 0.00 -> 19.1 mm
Other:
- board size 100 x 70 mm -> 130 x 66 mm
- net class Default: trace_width 1 -> 3
