File: 5V_supply/5V_supply.sch (KiCad schematic (older format))
At the start: 11 parts, among them J1 Conn_01x01, J2 Conn_01x01, J3 Conn_01x01, J4 Conn_01x01, J5 Conn_01x01, J6 Conn_01x01, J7 Conn_01x01, J8 Conn_01x01

Commit message: power supply finished
Parts:
- removed C1: 0,47x630V, Capacitor_THT:C_Rect_L33.0mm_W15.0mm_P27.50mm_MKS4, symbol Device:C
- removed C2: 0,1, Capacitor_THT:C_Rect_L7.0mm_W3.5mm_P5.00mm, symbol Device:C
- added F1: Fuse, Fuse:Fuseholder_Cylinder-5x20mm_Schurter_0031_8201_Horizontal_Open, symbol Device:Fuse
- added J10, J11, J12, J13, J9: Conn_01x01, Connector_Wire:SolderWirePad_1x01_Drill2.5mm, symbol Connector_Generic:Conn_01x01
Connections:
- net at J1.1 (Pin_1): now also F1.2; no longer J3.1 (Pin_1)
- net at C3.1, J7.1 (Pin_1): now also J11.1 (Pin_1); no longer J5.1 (Pin_1)
- net at C3.2, J8.1 (Pin_1): now also J13.1 (Pin_1); no longer J6.1 (Pin_1)
- new net: F1.1, J3.1 (Pin_1)
- new net: J5.1 (Pin_1), J9.1 (Pin_1)
- new net: J10.1 (Pin_1), J6.1 (Pin_1)
Other:
- note added: "filter"
- moved on the sheet: C3, J7, J8
Changed lines of the file:
@@
 AC_IN
-$Comp
-L Device:C C1
-U 1 1 5DDB012E
-P 2200 1700
-F 0 "C1" H 2315 1746 50  0000 L CNN
-F 1 "0,47x630V" H 2050 1300 50  0000 L CNN
-F 2 "Capacitor_THT:C_Rect_L33.0mm_W15.0mm_P27.50mm_MKS4" H 2238 1550 50  0001 C CNN
-F 3 "~" H 2200 1700 50  0001 C CNN
-	1    2200 1700
-	1    0    0    -1
-$EndComp
 $Comp
 L Connector_Generic:Conn_01x01 J3
@@
 -
 $Comp
-L Device:C C2
-U 1 1 5DDB04BE
-P 4250 1700
-F 0 "C2" H 4365 1746 50  0000 L CNN
-F 1 "0,1" H 4350 1650 50  0000 L CNN
-F 2 "Capacitor_THT:C_Rect_L7.0mm_W3.5mm_P5.00mm" H 4288 1550 50  0001 C CNN
-F 3 "~" H 4250 1700 50  0001 C CNN
-	1    4250 1700
-	1    0    0    -1
-$EndComp
-$Comp
 L Connector_Generic:Conn_01x01 J7
 U 1 1 5DDB054F
-P 5300 1450
-F 0 "J7" H 5219 1225 50  0000 C CNN
-F 1 "Conn_01x01" H 5219 1316 50  0000 C CNN
-F 2 "Connector_Wire:SolderWirePad_1x01_Drill2mm" H 5300 1450 50  0001 C CNN
-F 3 "~" H 5300 1450 50  0001 C CNN
-	1    5300 1450
+P 6950 1450
+F 0 "J7" H 6869 1225 50  0000 C CNN
+F 1 "Conn_01x01" H 6869 1316 50  0000 C CNN
+F 2 "Connector_Wire:SolderWirePad_1x01_Drill2mm" H 6950 1450 50  0001 C CNN
+F 3 "~" H 6950 1450 50  0001 C CNN
+	1    6950 1450
 	1    0    0    1
 $EndComp
@@
 L Connector_Generic:Conn_01x01 J8
 U 1 1 5DDB059D
-P 5300 1950
-F 0 "J8" H 5219 1725 50  0000 C CNN
-F 1 "Conn_01x01" H 5219 1816 50  0000 C CNN
-F 2 "Connector_Wire:SolderWirePad_1x01_Drill2mm" H 5300 1950 50  0001 C CNN
-F 3 "~" H 5300 1950 50  0001 C CNN
-	1    5300 1950
+P 6950 1950
+F 0 "J8" H 6869 1725 50  0000 C CNN
+F 1 "Conn_01x01" H 6869 1816 50  0000 C CNN
+F 2 "Connector_Wire:SolderWirePad_1x01_Drill2mm" H 6950 1950 50  0001 C CNN
+F 3 "~" H 6950 1950 50  0001 C CNN
+	1    6950 1950
 	1    0    0    1
 $EndComp
 Wire Wire Line
-	1800 1450 2200 1450
-Wire Wire Line
-	2650 1950 2200 1950
-Wire Wire Line
-	2200 1850 2200 1950
-Connection ~ 2200 1950
-Wire Wire Line
-	2200 1950 1800 1950
-Wire Wire Line
-	2200 1450 2200 1550
-Connection ~ 2200 1450
-Wire Wire Line
-	2200 1450 2650 1450
-Wire Wire Line
-	4000 1450 4250 1450
-Wire Wire Line
-	5100 1950 4700 1950
-Wire Wire Line
-	4250 1850 4250 1950
-Connection ~ 4250 1950
-Wire Wire Line
-	4250 1950 4000 1950
-Wire Wire Line
-	4250 1550 4250 1450
-Connection ~ 4250 1450
-Wire Wire Line
-	4250 1450 4700 1450
+	6750 1950 6350 1950
 Wire Notes Line
 	4150 2100 4150 1150
@@
 L Device:CP C3
 U 1 1 5DDB0A82
-P 4700 1700
-F 0 "C3" H 4818 1746 50  0000 L CNN
-F 1 "CP" H 4818 1655 50  0000 L CNN
-F 2 "Capacitor_THT:CP_Radial_D13.0mm_P7.50mm" H 4738 1550 50  0001 C CNN
-F 3 "~" H 4700 1700 50  0001 C CNN
-	1    4700 1700
+P 6350 1700
+F 0 "C3" H 6468 1746 50  0000 L CNN
+F 1 "CP" H 6468 1655 50  0000 L CNN
+F 2 "Capacitor_THT:CP_Radial_D13.0mm_P7.50mm" H 6388 1550 50  0001 C CNN
+F 3 "~" H 6350 1700 50  0001 C CNN
+	1    6350 1700
 	1    0    0    -1
 $EndComp
 Wire Wire Line
-	4700 1550 4700 1450
-Connection ~ 4700 1450
+	6350 1550 6350 1450
+Connection ~ 6350 1450
 Wire Wire Line
-	4700 1450 5100 1450
+	6350 1450 6750 1450
 Wire Wire Line
-	4700 1850 4700 1950
-Connection ~ 4700 1950
+	6350 1850 6350 1950
+Connection ~ 6350 1950
 Wire Wire Line
-	4700 1950 4250 1950
+	1800 1450 1950 1450
+Wire Wire Line
+	1800 1950 2650 1950
+Wire Notes Line
+	4350 1150 5450 1150
+Wire Notes Line
+	5450 1150 5450 2100
+Wire Notes Line
+	5450 2100 4350 2100
+Wire Notes Line
+	4350 2100 4350 1150
+$Comp
+L Connector_Generic:Conn_01x01 J11
+U 1 1 5DE03A99
+P 5150 1450
+F 0 "J11" H 5070 1225 50  0000 C CNN
+F 1 "Conn_01x01" H 5070 1316 50  0000 C CNN
+F 2 "Connector_Wire:SolderWirePad_1x01_Drill2.5mm" H 5150 1450 50  0001 C CNN
+F 3 "~" H 5150 1450 50  0001 C CNN
+	1    5150 1450
+	-1   0    0    1
+$EndComp
+$Comp
+L Connector_Generic:Conn_01x01 J12
+U 1 1 5DE03B25
+P 5150 1700
+F 0 "J12" H 5070 1475 50  0000 C CNN
+F 1 "Conn_01x01" H 5070 1566 50  0000 C CNN
+F 2 "Connector_Wire:SolderWirePad_1x01_Drill2.5mm" H 5150 1700 50  0001 C CNN
+F 3 "~" H 5150 1700 50  0001 C CNN
+	1    5150 1700
+	-1   0    0    1
+$EndComp
+$Comp
+L Connector_Generic:Conn_01x01 J13
+U 1 1 5DE03B51
+P 5150 1950
+F 0 "J13" H 5070 1725 50  0000 C CNN
+F 1 "Conn_01x01" H 5070 1816 50  0000 C CNN
+F 2 "Connector_Wire:SolderWirePad_1x01_Drill2.5mm" H 5150 1950 50  0001 C CNN
+F 3 "~" H 5150 1950 50  0001 C CNN
+	1    5150 1950
+	-1   0    0    1
+$EndComp
+$Comp
+L Connector_Generic:Conn_01x01 J9
+U 1 1 5DE03B8B
+P 4700 1450
+F 0 "J9" H 4619 1225 50  0000 C CNN
+F 1 "Conn_01x01" H 4619 1316 50  0000 C CNN
+F 2 "Connector_Wire:SolderWirePad_1x01_Drill2.5mm" H 4700 1450 50  0001 C CNN
+F 3 "~" H 4700 1450 50  0001 C CNN
+	1    4700 1450
+	1    0    0    1
+$EndComp
+$Comp
+L Connector_Generic:Conn_01x01 J10
+U 1 1 5DE03BD9
+P 4700 1950
+F 0 "J10" H 4619 1725 50  0000 C CNN
+F 1 "Conn_01x01" H 4619 1816 50  0000 C CNN
+F 2 "Connector_Wire:SolderWirePad_1x01_Drill2.5mm" H 4700 1950 50  0001 C CNN
+F 3 "~" H 4700 1950 50  0001 C CNN
+	1    4700 1950
+	1    0    0    1
+$EndComp
+Wire Wire Line
+	4500 1450 4000 1450
+Wire Wire Line
+	4000 1950 4500 1950
+Wire Wire Line
+	5350 1450 6350 1450
+Wire Wire Line
+	5350 1950 6350 1950
+Text Notes 4800 1250 0    50   ~ 0
+filter
+$Comp
+L Device:Fuse F1
+U 1 1 5DE04162
+P 2100 1450
+F 0 "F1" V 1903 1450 50  0000 C CNN
+F 1 "Fuse" V 1994 1450 50  0000 C CNN
+F 2 "Fuse:Fuseholder_Cylinder-5x20mm_Schurter_0031_8201_Horizontal_Open" V 2030 1450 50  0001 C CNN
+F 3 "~" H 2100 1450 50  0001 C CNN
+	1    2100 1450
+	0    1    1    0
+$EndComp
+Wire Wire Line
+	2250 1450 2650 1450
 $EndSCHEMATC
